File: PCB Files/ESP32/ESP32.kicad_sch (KiCad schematic)
At the start: 43 parts, among them J1 Conn_01x03_Pin, J11 Conn_01x05_Pin, J12 Conn_01x04_Pin, J13 Conn_01x04_Pin, J14 Conn_01x04_Pin, J15 Conn_01x04_Pin, J16 Conn_01x04_Pin, J2 Conn_01x03_Pin, J3 Conn_01x03_Pin, J4 Conn_01x03_Pin, J5 Conn_01x03_Pin, P1 USB_C_Plug_USB2.0, SW1 SW_Push, SW2 SW_Push, SW3 SW_Push, SW4 SW_Push, U1 ESP32-S3-WROOM-1, U2 AMS1117-3.3, U3 LM2596S-5

Commit message: updated PCB
Parts:
- removed C4: 100nF, Capacitor_SMD:C_0805_2012Metric_Pad1.18x1.45mm_HandSolder, symbol Device:C
- removed D3: D_Schottky, Diode_SMD:D_SMA, symbol Device:D_Schottky
- removed P1: USB_C_Plug_USB2.0, Connector_USB:USB_C_Receptacle_GCT_USB4085, symbol Connector:USB_C_Plug_USB2.0
- added J6: Conn_01x05_Pin, Connector_PinHeader_2.54mm:PinHeader_1x05_P2.54mm_Vertical, symbol Connector:Conn_01x05_Pin
- added J7: Conn_ARM_JTAG_SWD_10, Connector_PinHeader_1.27mm:PinHeader_2x05_P1.27mm_Vertical, symbol Connector:Conn_ARM_JTAG_SWD_10
- added JP1, JP2: SolderJumper_2_Open, Jumper:SolderJumper-2_P1.3mm_Open_RoundedPad1.0x1.5mm, symbol Jumper:SolderJumper_2_Open
- added Q1, Q2: SS8050, Package_TO_SOT_SMD:SOT-23, symbol Transistor_BJT:SS8050
- added R8, R9: 10k, Resistor_SMD:R_0805_2012Metric_Pad1.20x1.40mm_HandSolder, symbol Device:R
- BT1: footprint Connector_JST:JST_XH_B2B-XH-A_1x02_P2.50mm_Vertical -> Connector_PinHeader_2.54mm:PinHeader_1x02_P2.54mm_Vertical
- R2: value 5.1k -> 10k
- R3: value 1M -> 10k
- TP1, TP2: footprint TestPoint:TestPoint_THTPad_2.0x2.0mm_Drill1.0mm -> Connector_PinHeader_2.54mm:PinHeader_1x01_P2.54mm_Vertical
Connections:
- net +3.3V: now also J7.1 (VTref), JP2.2 (B); no longer C2.1, U2.2 (VO)
- net +5V: now also JP1.2 (B); no longer D2.1 (K)
- net 21: now also J3.2 (Pin_2)
- net 38: no longer J5.2 (Pin_2)
- net 47: now also J4.2 (Pin_2)
- net 48: now also J5.2 (Pin_2)
- net ADC2: now also J1.2 (Pin_2)
- net ADC8: now also J2.2 (Pin_2)
- net GND: now also J6.1 (Pin_1), J7.3 (GND), J7.5 (GND), J7.9 (GNDDetect); no longer R2.2, R3.2
- net RX: now also J6.3 (Pin_3)
- net TX: now also J6.2 (Pin_2)
- net EN: now reaches C1.2, R1.2, SW2.1, U1.3 (EN)
- net EN: now also J7.10 (~{RESET}), R8.2
- net RTS: now reaches R3.1
- net RTS: now also J6.4 (Pin_4), Q1.2 (E)
- net IO0: now reaches R4.1, SW1.1, U1.27 (IO0)
- net IO0: now also R9.2
- net DTR: now reaches R2.1
- net DTR: now also J6.5 (Pin_5), Q2.3 (C)
- net 39 renamed IO39
- net IO39: now also J7.4 (SWCLK/TCK); no longer J4.2 (Pin_2)
- net 40 renamed IO40
- net IO40: now also J7.6 (SWO/TDO); no longer J3.2 (Pin_2)
- net 41 renamed IO41
- net IO41: now also J7.8 (NC/TDI); no longer J2.2 (Pin_2)
- net 42 renamed IO42
- net IO42: now also J7.2 (SWDIO/TMS); no longer J1.2 (Pin_2)
- new net: C2.1, JP2.1 (A), U2.2 (VO)
- new net: Q1.1 (B), R2.2
- new net: Q1.3 (C), R8.1
- new net: Q2.2 (E), R9.1
- new net: Q2.1 (B), R3.2
- new net: D2.1 (K), JP1.1 (A)
Other:
- note removed: "USBC MODULE"
